File: OV9281/_saved_OV9281.sch (KiCad schematic (older format))
At the start: 72 parts, among them IC1 TLV73328PDBVT, IC2 TLV73318PDBVT, IC3 TLV73312PDBVT, J3 WE_68715014522, Q1 BSS138AKA, U1 OV9281, U2 OV9281, U3 NTS0104BQ, U4 NTB0104BQ, Y1 Farnell_1842027, Y2 Farnell_1842027

Commit message: PCB routing
Parts:
- C1, C2, C3: symbol antmicro_Capacitors_misc:C_4u7_0805 -> OV9281-rescue:C_4u7_0805-antmicro_Capacitors_misc
- C10, C12, C13, C18, C19, C21, C22, C24, C25, C27, C28, C33, C34, C35, C36, C38, C4, C5, C6, C7, C8: symbol antmicro_Capacitors_0603:C_1u_0603 -> OV9281-rescue:C_1u_0603-antmicro_Capacitors_0603
- C14, C15, C16, C17, C20, C23, C29, C30, C31, C32, C37, C9: symbol antmicro_Capacitors_0402:C_100n_0402_6V3 -> OV9281-rescue:C_100n_0402_6V3-antmicro_Capacitors_0402
- IC1: symbol antmicro_PMIC_Voltage_Regulators_Linear:TLV73328PDBVT -> OV9281-rescue:TLV73328PDBVT-antmicro_PMIC_Voltage_Regulators_Linear
- IC2: symbol antmicro_PMIC_Voltage_Regulators_Linear:TLV73318PDBVT -> OV9281-rescue:TLV73318PDBVT-antmicro_PMIC_Voltage_Regulators_Linear
- IC3: symbol antmicro_PMIC_Voltage_Regulators_Linear:TLV73312PDBVT -> OV9281-rescue:TLV73312PDBVT-antmicro_PMIC_Voltage_Regulators_Linear
- J3: symbol antmicro_FCC_Connectors:WE_68715014522 -> OV9281-rescue:WE_68715014522-antmicro_FCC_Connectors
- L1, L2, L3, L4, L5, L6: symbol antmicro_Fixed_Inductors:MLP2012S3R3MT -> OV9281-rescue:MLP2012S3R3MT-antmicro_Fixed_Inductors
- Q1: symbol antmicro_Transistors_FETs_MOSFETs_Single:BSS138AKA -> OV9281-rescue:BSS138AKA-antmicro_Transistors_FETs_MOSFETs_Single
- R1, R2, R3, R4: symbol antmicro_Resistors_0402:R_2k37_0402 -> OV9281-rescue:R_2k37_0402-antmicro_Resistors_0402
- R10, R11, R13, R14, R15, R16, R17, R20, R21, R5, R7, R8, R9: symbol antmicro_Resistors_0402:R_0R_0402 -> OV9281-rescue:R_0R_0402-antmicro_Resistors_0402
- R18: symbol antmicro_Resistors_0402:R_10k_0402 -> OV9281-rescue:R_10k_0402-antmicro_Resistors_0402
- R19: symbol antmicro_Resistors_0402:R_2k_0402 -> OV9281-rescue:R_2k_0402-antmicro_Resistors_0402
- U1, U2: symbol antmicro_Image_Sensors:OV9281 -> OV9281-rescue:OV9281-antmicro_Image_Sensors
- U3: symbol antmicro_Logic_Translators_Level_Shifters:NTS0104BQ -> OV9281-rescue:NTS0104BQ-antmicro_Logic_Translators_Level_Shifters
- U4: symbol antmicro_Logic_Translators_Level_Shifters:NTB0104BQ -> OV9281-rescue:NTB0104BQ-antmicro_Logic_Translators_Level_Shifters
- Y1, Y2: symbol antmicro_Oscillators:Farnell_1842027 -> OV9281-rescue:Farnell_1842027-antmicro_Oscillators
