File: OV9281-Dual-Camera_Board-Rev.1.1/OV9281-Dual-Camera-Board-Rev.1.1.kicad_pcb (KiCad board)
At the start: 4 copper layers, 100 x 25 mm, 80 parts, among them IC1 TLV73328PDBVT, IC2 TLV73318PDBVT, IC3 TLV73312PDBVT, J3 WE_68715014522, Q1 BSS138AKA, U1 OV9281, U2 OV9281, U3 NTS0104BQ, U4 NTB0104BQ, Y1 7C-24.000MBB-T, Y2 7C-24.000MBB-T

Commit message: Cleanup
Parts:
- C1, C2, C3: footprint antmicro-footprints:0805-cap -> OV9281-Dual-Camera-Board-Rev.1.1-footprints:0805-cap
- C10, C12, C13, C18, C19, C21, C22, C24, C25, C27, C28, C33, C34, C35, C36, C38, C4, C5, C6, C7, C8: footprint antmicro-footprints:0603-cap -> OV9281-Dual-Camera-Board-Rev.1.1-footprints:0603-cap
- C14, C15, C16, C17, C20, C23, C29, C30, C31, C32, C37, C9: footprint antmicro-footprints:0402-cap -> OV9281-Dual-Camera-Board-Rev.1.1-footprints:0402-cap
- IC1, IC2, IC3: footprint antmicro-footprints:SOT-23-5 -> OV9281-Dual-Camera-Board-Rev.1.1-footprints:SOT-23-5
- J3: footprint antmicro-footprints:WE_68715014522 -> OV9281-Dual-Camera-Board-Rev.1.1-footprints:WE_68715014522
- L1, L2, L3, L4, L5, L6: footprint antmicro-footprints:0805-res -> OV9281-Dual-Camera-Board-Rev.1.1-footprints:0805-res
- MP1, MP2, MP3, MP4: footprint antmicro-footprints:9774030243R -> OV9281-Dual-Camera-Board-Rev.1.1-footprints:9774030243R
- N1: footprint antmicro-footprints:antmicro-logo_scaled_20mm -> OV9281-Dual-Camera-Board-Rev.1.1-footprints:antmicro-logo_scaled_20mm
- Q1: footprint antmicro-footprints:SOT-23-3 -> OV9281-Dual-Camera-Board-Rev.1.1-footprints:SOT-23-3
- R1, R10, R11, R12, R13, R14, R15, R16, R17, R18, R19, R2, R20, R21, R22, R3, R4, R5, R6, R7, R8, R9: footprint antmicro-footprints:0402-res -> OV9281-Dual-Camera-Board-Rev.1.1-footprints:0402-res
- U1, U2: footprint antmicro-footprints:ov9281 -> OV9281-Dual-Camera-Board-Rev.1.1-footprints:ov9281
- U3, U4: footprint antmicro-footprints:QDHVQFN14 -> OV9281-Dual-Camera-Board-Rev.1.1-footprints:QDHVQFN14
- Y1, Y2: value 7C-24.000MBB-T -> Farnell_1842027; footprint antmicro-footprints:7C-24.000MBB-T -> OV9281-Dual-Camera-Board-Rev.1.1-footprints:7C-24.000MBB-T
