File: OV9281-Dual-Camera_Board-Rev.1.1/OV9281-Dual-Camera-Board-Rev.1.1.sch (KiCad schematic (older format))
At the start: 80 parts, among them IC1 TLV73328PDBVT, IC2 TLV73318PDBVT, IC3 TLV73312PDBVT, J3 WE_68715014522, Q1 BSS138AKA, U1 OV9281, U2 OV9281, U3 NTS0104BQ, U4 NTB0104BQ, Y1 7C-24.000MBB-T, Y2 7C-24.000MBB-T

Commit message: Cleanup
Parts:
- C1, C2, C3: footprint antmicro-footprints:0805-cap -> OV9281-Dual-Camera-Board-Rev.1.1-footprints:0805-cap; symbol antmicroCapacitorsmisc:C_4u7_0805 -> OV9281-Dual-Camera-Board-Rev.1.1:C_4u7_0805
- C10, C12, C13, C18, C19, C21, C22, C24, C25, C27, C28, C33, C34, C35, C36, C38, C4, C5, C6, C7, C8: footprint antmicro-footprints:0603-cap -> OV9281-Dual-Camera-Board-Rev.1.1-footprints:0603-cap; symbol antmicroCapacitors0603:C_1u_0603 -> OV9281-Dual-Camera-Board-Rev.1.1:C_1u_0603
- C14, C15, C16, C17, C20, C23, C29, C30, C31, C32, C37, C9: footprint antmicro-footprints:0402-cap -> OV9281-Dual-Camera-Board-Rev.1.1-footprints:0402-cap; symbol antmicroCapacitors0402:C_100n_0402_6V3 -> OV9281-Dual-Camera-Board-Rev.1.1:C_100n_0402_6V3
- IC1: footprint antmicro-footprints:SOT-23-5 -> OV9281-Dual-Camera-Board-Rev.1.1-footprints:SOT-23-5; symbol antmicroPMICVoltageRegulatorsLinear:TLV73328PDBVT -> OV9281-Dual-Camera-Board-Rev.1.1:TLV73328PDBVT
- IC2: footprint antmicro-footprints:SOT-23-5 -> OV9281-Dual-Camera-Board-Rev.1.1-footprints:SOT-23-5; symbol antmicroPMICVoltageRegulatorsLinear:TLV73318PDBVT -> OV9281-Dual-Camera-Board-Rev.1.1:TLV73318PDBVT
- IC3: footprint antmicro-footprints:SOT-23-5 -> OV9281-Dual-Camera-Board-Rev.1.1-footprints:SOT-23-5; symbol antmicroPMICVoltageRegulatorsLinear:TLV73312PDBVT -> OV9281-Dual-Camera-Board-Rev.1.1:TLV73312PDBVT
- J3: footprint antmicro-footprints:WE_68715014522 -> OV9281-Dual-Camera-Board-Rev.1.1-footprints:WE_68715014522; symbol antmicroFCCConnectors:WE_68715014522 -> OV9281-Dual-Camera-Board-Rev.1.1:WE_68715014522
- L1, L2, L3, L4, L5, L6: footprint antmicro-footprints:0805-res -> OV9281-Dual-Camera-Board-Rev.1.1-footprints:0805-res; symbol antmicroFixedInductors:MLP2012S3R3MT -> OV9281-Dual-Camera-Board-Rev.1.1:MLP2012S3R3MT
- MP1, MP2, MP3, MP4: footprint antmicro-footprints:9774030243R -> OV9281-Dual-Camera-Board-Rev.1.1-footprints:9774030243R; symbol antmicroMechanicalParts:PCB_Spacer_M2 -> OV9281-Dual-Camera-Board-Rev.1.1:PCB_Spacer_M2
- N1: footprint antmicro-footprints:antmicro-logo_scaled_20mm -> OV9281-Dual-Camera-Board-Rev.1.1-footprints:antmicro-logo_scaled_20mm; symbol antmicroMechanicalParts:antmicro_logo -> OV9281-Dual-Camera-Board-Rev.1.1:antmicro_logo
- Q1: footprint antmicro-footprints:SOT-23-3 -> OV9281-Dual-Camera-Board-Rev.1.1-footprints:SOT-23-3; symbol antmicroTransistorsFETsMOSFETsSingle:BSS138AKA -> OV9281-Dual-Camera-Board-Rev.1.1:BSS138AKA
- R1, R2, R3, R4: footprint antmicro-footprints:0402-res -> OV9281-Dual-Camera-Board-Rev.1.1-footprints:0402-res; symbol antmicroResistors0402:R_2k37_0402 -> OV9281-Dual-Camera-Board-Rev.1.1:R_2k37_0402
- R10, R11, R12, R13, R14, R15, R16, R17, R20, R21, R22, R5, R6, R7, R8, R9: footprint antmicro-footprints:0402-res -> OV9281-Dual-Camera-Board-Rev.1.1-footprints:0402-res; symbol antmicroResistors0402:R_0R_0402 -> OV9281-Dual-Camera-Board-Rev.1.1:R_0R_0402
- R18: footprint antmicro-footprints:0402-res -> OV9281-Dual-Camera-Board-Rev.1.1-footprints:0402-res; symbol antmicroResistors0402:R_10k_0402 -> OV9281-Dual-Camera-Board-Rev.1.1:R_10k_0402
- R19: footprint antmicro-footprints:0402-res -> OV9281-Dual-Camera-Board-Rev.1.1-footprints:0402-res; symbol antmicroResistors0402:R_2k_0402 -> OV9281-Dual-Camera-Board-Rev.1.1:R_2k_0402
- U1, U2: footprint antmicro-footprints:ov9281 -> OV9281-Dual-Camera-Board-Rev.1.1-footprints:ov9281; symbol antmicroImageSensors:OV9281 -> OV9281-Dual-Camera-Board-Rev.1.1:OV9281
- U3: footprint antmicro-footprints:QDHVQFN14 -> OV9281-Dual-Camera-Board-Rev.1.1-footprints:QDHVQFN14; symbol antmicroLogicTranslatorsLevelShifters:NTS0104BQ -> OV9281-Dual-Camera-Board-Rev.1.1:NTS0104BQ
- U4: footprint antmicro-footprints:QDHVQFN14 -> OV9281-Dual-Camera-Board-Rev.1.1-footprints:QDHVQFN14; symbol antmicroLogicTranslatorsLevelShifters:NTB0104BQ -> OV9281-Dual-Camera-Board-Rev.1.1:NTB0104BQ
- Y1, Y2: footprint antmicro-footprints:7C-24.000MBB-T -> OV9281-Dual-Camera-Board-Rev.1.1-footprints:7C-24.000MBB-T; symbol antmicroOscillators:7C-24.000MBB-T -> OV9281-Dual-Camera-Board-Rev.1.1:7C-24.000MBB-T
Connections:
- wire segments 399 -> 398
Other:
- note added: "Camera #1"
- note added: "Camera #2"
- note added: "Clk_Cam#1\n"
- note added: "Clk_Cam#2\n"
- note added: "Mode select"
- note added: "OV9281 sensors"
- note added: "Place close to sensors"
- note added: "Power Supply"
- note added: "Standoffs"
- note removed: "CLK_Cam #1\n"
- note removed: "CLK_Cam #2\n"
- note removed: "Camera syncs tied with each other"
- note removed: "OV9281 Camera #1"
- note removed: "OV9281 Camera #2"
- note removed: "Voltage Regulators"
- note removed: "analog and digital grounds connected in signle point"
