File: OV9281-Dual-Camera-Board.kicad_pcb (KiCad board)
At the start: 4 copper layers, 100 x 25 mm, 83 parts, among them IC1 TLV73328PDBVT, IC2 TLV73318PDBVT, IC3 TLV73312PDBVT, J3 WE_68715014522, Q1 BSS138AKA, U1 OV9281, U2 OV9281, U3 NTS0104BQ, U4 NTB0104BQ, Y1 Farnell_1842027, Y2 Farnell_1842027

Commit message: Updated project structure
Parts:
- MP5, MP6: footprint antmicro-footprints:Camera_Lens_20mm -> OV9281-Dual-Camera-Board-footprints:Camera_Lens_20mm
- N2: footprint antmicro-footprints:oshw-logo -> OV9281-Dual-Camera-Board-footprints:oshw-logo
Changed lines of the file:
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@@
     )
   )
-  (module antmicro-footprints:Camera_Lens_20mm (layer B.Cu)
+  (module OV9281-Dual-Camera-Board-footprints:Camera_Lens_20mm (layer B.Cu)
     (at 185 112.5)
     (fp_text reference MP6 (at -6.7 9.5) (layer B.SilkS)
@@
     (pad 2 thru_hole circle (at -10 0) (size 1.5 1.5) (drill 1.5) (layers *.Cu *.Mask))
     (pad 1 thru_hole circle (at 10 0) (size 1.5 1.5) (drill 1.5) (layers *.Cu *.Mask))
-    (model ${ANT3DMDL}/Assembled_Lens.step
+    (model ${KIPRJMOD}/lib/3d-models/Assembled_Lens.step
       (at (xyz 0 0 0))
       (scale (xyz 1 1 1))
@@
     )
   )
-  (module antmicro-footprints:Camera_Lens_20mm (layer B.Cu)
+  (module OV9281-Dual-Camera-Board-footprints:Camera_Lens_20mm (layer B.Cu)
     (at 115 112.5)
     (fp_text reference MP5 (at -6.7 9.5) (layer B.SilkS)
@@
     (pad 2 thru_hole circle (at -10 0) (size 1.5 1.5) (drill 1.5) (layers *.Cu *.Mask))
     (pad 1 thru_hole circle (at 10 0) (size 1.5 1.5) (drill 1.5) (layers *.Cu *.Mask))
-    (model ${ANT3DMDL}/Assembled_Lens.step
+    (model ${KIPRJMOD}/lib/3d-models/Assembled_Lens.step
       (at (xyz 0 0 0))
       (scale (xyz 1 1 1))
@@
     )
   )
-  (module antmicro-footprints:oshw-logo (layer F.Cu)
+  (module OV9281-Dual-Camera-Board-footprints:oshw-logo (layer F.Cu)
     (at 150 108)
     (fp_text reference N2 (at -3.08 -4.76) (layer F.SilkS) hide
