File: OV9281-Dual-Camera-Board.sch (KiCad schematic (older format))
At the start: 80 parts, among them IC1 TLV73328PDBVT, IC2 TLV73318PDBVT, IC3 TLV73312PDBVT, J3 WE_68715014522, Q1 BSS138AKA, U1 OV9281, U2 OV9281, U3 NTS0104BQ, U4 NTB0104BQ, Y1 7C-24.000MBB-T, Y2 7C-24.000MBB-T

Commit message: Added OSHW logo, updated hole spacing for lens mount
Parts:
- added MP5, MP6: Camera_Lens, antmicro-footprints:Camera_Lens_20mm, symbol antmicroCameramodules:Camera_Lens
- added N2: oshw_logo, antmicro-footprints:oshw-logo, symbol antmicroMechanicalParts:oshw_logo
Other:
- note added: "Camera Lenses"
- note added: "Logos"
- moved on the sheet: J3, MP1, MP2, MP3, MP4, R1, R2, R3, R4, R5, U3, U4

Commit message: Updated project structure
Parts:
- MP5, MP6: footprint antmicro-footprints:Camera_Lens_20mm -> OV9281-Dual-Camera-Board-footprints:Camera_Lens_20mm; symbol antmicroCameramodules:Camera_Lens -> OV9281-Dual-Camera-Board:Camera_Lens
- N2: footprint antmicro-footprints:oshw-logo -> OV9281-Dual-Camera-Board-footprints:oshw-logo; symbol antmicroMechanicalParts:oshw_logo -> OV9281-Dual-Camera-Board:oshw_logo
Changed lines of the file:
@@
 $EndBitmap
 $Comp
-L antmicroMechanicalParts:oshw_logo N2
+L OV9281-Dual-Camera-Board:oshw_logo N2
 U 1 1 5ECAD722
 P 15000 7050
 F 0 "N2" H 14900 7100 50  0000 L CNN
 F 1 "oshw_logo" H 14850 6900 50  0000 L CNN
-F 2 "antmicro-footprints:oshw-logo" H 15020 6810 50  0001 C CNN
+F 2 "OV9281-Dual-Camera-Board-footprints:oshw-logo" H 15020 6810 50  0001 C CNN
 F 3 "" H 15000 7050 50  0001 C CNN
 	1    15000 7050
@@
 Logos
 $Comp
-L antmicroCameramodules:Camera_Lens MP6
+L OV9281-Dual-Camera-Board:Camera_Lens MP6
 U 1 1 5E7B1125
 P 13700 7100
 F 0 "MP6" H 14028 7153 59  0000 L CNN
 F 1 "Camera_Lens" H 14028 7048 59  0000 L CNN
-F 2 "antmicro-footprints:Camera_Lens_20mm" H 15600 7150 118 0001 C CNN
+F 2 "OV9281-Dual-Camera-Board-footprints:Camera_Lens_20mm" H 15600 7150 118 0001 C CNN
 F 3 "" H 13700 7100 118 0001 C CNN
 F 4 "" H 14028 7041 50  0000 L CNN "MPN"
@@
 $EndComp
 $Comp
-L antmicroCameramodules:Camera_Lens MP5
+L OV9281-Dual-Camera-Board:Camera_Lens MP5
 U 1 1 5E7B7776
 P 12400 7100
 F 0 "MP5" H 12728 7153 59  0000 L CNN
 F 1 "Camera_Lens" H 12728 7048 59  0000 L CNN
-F 2 "antmicro-footprints:Camera_Lens_20mm" H 14300 7150 118 0001 C CNN
+F 2 "OV9281-Dual-Camera-Board-footprints:Camera_Lens_20mm" H 14300 7150 118 0001 C CNN
 F 3 "" H 12400 7100 118 0001 C CNN
 F 4 "" H 12728 7041 50  0000 L CNN "MPN"
